Commit message: Refactor folder structure to follow ros conventions
Signed-off-by: Baoan Du <baoan.du.xj@renesas.com>

File: urdf/reference/ruihand6_left_ref.urdf (robot description, URDF)
Before this commit: robot ruihand6z, 17 links, 16 joints
Links:
- link base_link: geometry collision mesh filename=package://ruiyan_rh2_hand_description/meshes/ruihand6z/base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; visual mesh filename=package://ruiyan_rh2_hand_description/meshes/ruihand6z/base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
- link fz11_Link: geometry collision mesh filename=package://ruiyan_rh2_hand_description/meshes/ruihand6z/fz11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; visual mesh filename=package://ruiyan_rh2_hand_description/meshes/ruihand6z/fz11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
- link fz12_Link: geometry collision mesh filename=package://ruiyan_rh2_hand_description/meshes/ruihand6z/fz12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; visual mesh filename=package://ruiyan_rh2_hand_description/meshes/ruihand6z/fz12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
- link fz13_Link: geometry collision mesh filename=package://ruiyan_rh2_hand_description/meshes/ruihand6z/fz13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; visual mesh filename=package://ruiyan_rh2_hand_description/meshes/ruihand6z/fz13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
- link fz14_Link: geometry collision mesh filename=package://ruiyan_rh2_hand_description/meshes/ruihand6z/fz14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; visual mesh filename=package://ruiyan_rh2_hand_description/meshes/ruihand6z/fz14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
- link fz21_Link: geometry collision mesh filename=package://ruiyan_rh2_hand_description/meshes/ruihand6z/fz21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; visual mesh filename=package://ruiyan_rh2_hand_description/meshes/ruihand6z/fz21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
- link fz22_Link: geometry collision mesh filename=package://ruiyan_rh2_hand_description/meshes/ruihand6z/fz22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; visual mesh filename=package://ruiyan_rh2_hand_description/meshes/ruihand6z/fz22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
- link fz23_Link: geometry collision mesh filename=package://ruiyan_rh2_hand_description/meshes/ruihand6z/fz23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; visual mesh filename=package://ruiyan_rh2_hand_description/meshes/ruihand6z/fz23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
- link fz31_Link: geometry collision mesh filename=package://ruiyan_rh2_hand_description/meshes/ruihand6z/fz31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; visual mesh filename=package://ruiyan_rh2_hand_description/meshes/ruihand6z/fz31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
- link fz32_Link: geometry collision mesh filename=package://ruiyan_rh2_hand_description/meshes/ruihand6z/fz32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; visual mesh filename=package://ruiyan_rh2_hand_description/meshes/ruihand6z/fz32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
- link fz33_Link: geometry collision mesh filename=package://ruiyan_rh2_hand_description/meshes/ruihand6z/fz33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; visual mesh filename=package://ruiyan_rh2_hand_description/meshes/ruihand6z/fz33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
- link fz41_Link: geometry collision mesh filename=package://ruiyan_rh2_hand_description/meshes/ruihand6z/fz41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; visual mesh filename=package://ruiyan_rh2_hand_description/meshes/ruihand6z/fz41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
- link fz42_Link: geometry collision mesh filename=package://ruiyan_rh2_hand_description/meshes/ruihand6z/fz42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; visual mesh filename=package://ruiyan_rh2_hand_description/meshes/ruihand6z/fz42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
- link fz43_Link: geometry collision mesh filename=package://ruiyan_rh2_hand_description/meshes/ruihand6z/fz43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; visual mesh filename=package://ruiyan_rh2_hand_description/meshes/ruihand6z/fz43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
- link fz51_Link: geometry collision mesh filename=package://ruiyan_rh2_hand_description/meshes/ruihand6z/fz51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; visual mesh filename=package://ruiyan_rh2_hand_description/meshes/ruihand6z/fz51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
- link fz52_Link: geometry collision mesh filename=package://ruiyan_rh2_hand_description/meshes/ruihand6z/fz52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; visual mesh filename=package://ruiyan_rh2_hand_description/meshes/ruihand6z/fz52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
- link fz53_Link: geometry collision mesh filename=package://ruiyan_rh2_hand_description/meshes/ruihand6z/fz53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; visual mesh filename=package://ruiyan_rh2_hand_description/meshes/ruihand6z/fz53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

File: urdf/reference/ruihand6_right_ref.urdf (robot description, URDF)
Before this commit: robot ruihand6y, 17 links, 16 joints
Links:
- link base_link: geometry collision mesh filename=package://ruiyan_rh2_hand_description/meshes/ruihand6y/base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; visual mesh filename=package://ruiyan_rh2_hand_description/meshes/ruihand6y/base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
- link fy11_Link: geometry collision mesh filename=package://ruiyan_rh2_hand_description/meshes/ruihand6y/fy11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; visual mesh filename=package://ruiyan_rh2_hand_description/meshes/ruihand6y/fy11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
- link fy12_Link: geometry collision mesh filename=package://ruiyan_rh2_hand_description/meshes/ruihand6y/fy12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; visual mesh filename=package://ruiyan_rh2_hand_description/meshes/ruihand6y/fy12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
- link fy13_Link: geometry collision mesh filename=package://ruiyan_rh2_hand_description/meshes/ruihand6y/fy13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; visual mesh filename=package://ruiyan_rh2_hand_description/meshes/ruihand6y/fy13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
- link fy14_Link: geometry collision mesh filename=package://ruiyan_rh2_hand_description/meshes/ruihand6y/fy14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; visual mesh filename=package://ruiyan_rh2_hand_description/meshes/ruihand6y/fy14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
- link fy21_Link: geometry collision mesh filename=package://ruiyan_rh2_hand_description/meshes/ruihand6y/fy21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; visual mesh filename=package://ruiyan_rh2_hand_description/meshes/ruihand6y/fy21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
- link fy22_Link: geometry collision mesh filename=package://ruiyan_rh2_hand_description/meshes/ruihand6y/fy22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; visual mesh filename=package://ruiyan_rh2_hand_description/meshes/ruihand6y/fy22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
- link fy23_Link: geometry collision mesh filename=package://ruiyan_rh2_hand_description/meshes/ruihand6y/fy23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; visual mesh filename=package://ruiyan_rh2_hand_description/meshes/ruihand6y/fy23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
- link fy31_Link: geometry collision mesh filename=package://ruiyan_rh2_hand_description/meshes/ruihand6y/fy31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; visual mesh filename=package://ruiyan_rh2_hand_description/meshes/ruihand6y/fy31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
- link fy32_Link: geometry collision mesh filename=package://ruiyan_rh2_hand_description/meshes/ruihand6y/fy32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; visual mesh filename=package://ruiyan_rh2_hand_description/meshes/ruihand6y/fy32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
- link fy33_Link: geometry collision mesh filename=package://ruiyan_rh2_hand_description/meshes/ruihand6y/fy33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; visual mesh filename=package://ruiyan_rh2_hand_description/meshes/ruihand6y/fy33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
- link fy41_Link: geometry collision mesh filename=package://ruiyan_rh2_hand_description/meshes/ruihand6y/fy41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; visual mesh filename=package://ruiyan_rh2_hand_description/meshes/ruihand6y/fy41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
- link fy42_Link: geometry collision mesh filename=package://ruiyan_rh2_hand_description/meshes/ruihand6y/fy42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; visual mesh filename=package://ruiyan_rh2_hand_description/meshes/ruihand6y/fy42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
- link fy43_Link: geometry collision mesh filename=package://ruiyan_rh2_hand_description/meshes/ruihand6y/fy43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; visual mesh filename=package://ruiyan_rh2_hand_description/meshes/ruihand6y/fy43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
- link fy51_Link: geometry collision mesh filename=package://ruiyan_rh2_hand_description/meshes/ruihand6y/fy51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; visual mesh filename=package://ruiyan_rh2_hand_description/meshes/ruihand6y/fy51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
- link fy52_Link: geometry collision mesh filename=package://ruiyan_rh2_hand_description/meshes/ruihand6y/fy52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; visual mesh filename=package://ruiyan_rh2_hand_description/meshes/ruihand6y/fy52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
- link fy53_Link: geometry collision mesh filename=package://ruiyan_rh2_hand_description/meshes/ruihand6y/fy53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; visual mesh filename=package://ruiyan_rh2_hand_description/meshes/ruihand6y/fy53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

File: urdf/ruiyan_hand_left_macro.xacro (robot description, xacro)
@@ -20,14 +20,14 @@
         <origin xyz="0 0 0" rpy="0 0 0"/>
         <geometry>
-          <mesh filename="package://ruiyan_rh2_hand_description/urdf/meshes/ruihand6z/base_link.STL"/>
-        </geometry>
-        <material name="">
-          <color rgba="0.898039215686275 0.917647058823529 0.929411764705882 1"/>
-        </material>
-      </visual>
-      <collision>
-        <origin xyz="0 0 0" rpy="0 0 0"/>
-        <geometry>
-          <mesh filename="package://ruiyan_rh2_hand_description/urdf/meshes/ruihand6z/base_link.STL"/>
+          <mesh filename="package://ruiyan_rh2_hand_description/meshes/ruihand6z/base_link.STL"/>
+        </geometry>
+        <material name="">
+          <color rgba="0.898039215686275 0.917647058823529 0.929411764705882 1"/>
+        </material>
+      </visual>
+      <collision>
+        <origin xyz="0 0 0" rpy="0 0 0"/>
+        <geometry>
+          <mesh filename="package://ruiyan_rh2_hand_description/meshes/ruihand6z/base_link.STL"/>
         </geometry>
       </collision>
@@ -44,14 +44,14 @@
         <origin xyz="0 0 0" rpy="0 0 0"/>
         <geometry>
-          <mesh filename="package://ruiyan_rh2_hand_description/urdf/meshes/ruihand6z/fz11_Link.STL"/>
-        </geometry>
-        <material name="">
-          <color rgba="0.898039215686275 0.917647058823529 0.929411764705882 1"/>
-        </material>
-      </visual>
-      <collision>
-        <origin xyz="0 0 0" rpy="0 0 0"/>
-        <geometry>
-          <mesh filename="package://ruiyan_rh2_hand_description/urdf/meshes/ruihand6z/fz11_Link.STL"/>
+          <mesh filename="package://ruiyan_rh2_hand_description/meshes/ruihand6z/fz11_Link.STL"/>
+        </geometry>
+        <material name="">
+          <color rgba="0.898039215686275 0.917647058823529 0.929411764705882 1"/>
+        </material>
+      </visual>
+      <collision>
+        <origin xyz="0 0 0" rpy="0 0 0"/>
+        <geometry>
+          <mesh filename="package://ruiyan_rh2_hand_description/meshes/ruihand6z/fz11_Link.STL"/>
         </geometry>
       </collision>
@@ -75,14 +75,14 @@
         <origin xyz="0 0 0" rpy="0 0 0"/>
         <geometry>
-          <mesh filename="package://ruiyan_rh2_hand_description/urdf/meshes/ruihand6z/fz12_Link.STL"/>
-        </geometry>
-        <material name="">
-          <color rgba="0.898039215686275 0.917647058823529 0.929411764705882 1"/>
-        </material>
-      </visual>
-      <collision>
-        <origin xyz="0 0 0" rpy="0 0 0"/>
-        <geometry>
-          <mesh filename="package://ruiyan_rh2_hand_description/urdf/meshes/ruihand6z/fz12_Link.STL"/>
+          <mesh filename="package://ruiyan_rh2_hand_description/meshes/ruihand6z/fz12_Link.STL"/>
+        </geometry>
+        <material name="">
+          <color rgba="0.898039215686275 0.917647058823529 0.929411764705882 1"/>
+        </material>
+      </visual>
+      <collision>
+        <origin xyz="0 0 0" rpy="0 0 0"/>
+        <geometry>
+          <mesh filename="package://ruiyan_rh2_hand_description/meshes/ruihand6z/fz12_Link.STL"/>
         </geometry>
       </collision>
@@ -106,14 +106,14 @@
         <origin xyz="0 0 0" rpy="0 0 0"/>
         <geometry>
-          <mesh filename="package://ruiyan_rh2_hand_description/urdf/meshes/ruihand6z/fz13_Link.STL"/>
-        </geometry>
-        <material name="">
-          <color rgba="0.898039215686275 0.917647058823529 0.929411764705882 1"/>
-        </material>
-      </visual>
-      <collision>
-        <origin xyz="0 0 0" rpy="0 0 0"/>
-        <geometry>
-          <mesh filename="package://ruiyan_rh2_hand_description/urdf/meshes/ruihand6z/fz13_Link.STL"/>
+          <mesh filename="package://ruiyan_rh2_hand_description/meshes/ruihand6z/fz13_Link.STL"/>
+        </geometry>
+        <material name="">
+          <color rgba="0.898039215686275 0.917647058823529 0.929411764705882 1"/>
+        </material>
+      </visual>
+      <collision>
+        <origin xyz="0 0 0" rpy="0 0 0"/>
+        <geometry>
+          <mesh filename="package://ruiyan_rh2_hand_description/meshes/ruihand6z/fz13_Link.STL"/>
         </geometry>
       </collision>
@@ -138,5 +138,5 @@
         <origin xyz="0 0 0" rpy="0 0 0"/>
         <geometry>
-          <mesh filename="package://ruiyan_rh2_hand_description/urdf/meshes/ruihand6z/fz14_Link.STL"/>
+          <mesh filename="package://ruiyan_rh2_hand_description/meshes/ruihand6z/fz14_Link.STL"/>
         </geometry>
         <material name="">
@@ -147,5 +147,5 @@
         <origin xyz="0 0 0" rpy="0 0 0"/>
         <geometry>
-          <mesh filename="package://ruiyan_rh2_hand_description/urdf/meshes/ruihand6z/fz14_Link.STL"/>
+          <mesh filename="package://ruiyan_rh2_hand_description/meshes/ruihand6z/fz14_Link.STL"/>
         </geometry>
       </collision>
@@ -169,14 +169,14 @@
         <origin xyz="0 0 0" rpy="0 0 0"/>
         <geometry>
-          <mesh filename="package://ruiyan_rh2_hand_description/urdf/meshes/ruihand6z/fz21_Link.STL"/>
-        </geometry>
-        <material name="">
-          <color rgba="0.898039215686275 0.917647058823529 0.929411764705882 1"/>
-        </material>
-      </visual>
-      <collision>
-        <origin xyz="0 0 0" rpy="0 0 0"/>
-        <geometry>
-          <mesh filename="package://ruiyan_rh2_hand_description/urdf/meshes/ruihand6z/fz21_Link.STL"/>
+          <mesh filename="package://ruiyan_rh2_hand_description/meshes/ruihand6z/fz21_Link.STL"/>
+        </geometry>
+        <material name="">
+          <color rgba="0.898039215686275 0.917647058823529 0.929411764705882 1"/>
+        </material>
+      </visual>
+      <collision>
+        <origin xyz="0 0 0" rpy="0 0 0"/>
+        <geometry>
+          <mesh filename="package://ruiyan_rh2_hand_description/meshes/ruihand6z/fz21_Link.STL"/>
         </geometry>
       </collision>
@@ -200,5 +200,5 @@
         <origin xyz="0 0 0" rpy="0 0 0"/>
         <geometry>
-          <mesh filename="package://ruiyan_rh2_hand_description/urdf/meshes/ruihand6z/fz22_Link.STL"/>
+          <mesh filename="package://ruiyan_rh2_hand_description/meshes/ruihand6z/fz22_Link.STL"/>
         </geometry>
         <material name="">
@@ -209,5 +209,5 @@
         <origin xyz="0 0 0" rpy="0 0 0"/>
         <geometry>
-          <mesh filename="package://ruiyan_rh2_hand_description/urdf/meshes/ruihand6z/fz22_Link.STL"/>
+          <mesh filename="package://ruiyan_rh2_hand_description/meshes/ruihand6z/fz22_Link.STL"/>
         </geometry>
       </collision>
@@ -232,5 +232,5 @@
         <origin xyz="0 0 0" rpy="0 0 0"/>
         <geometry>
-          <mesh filename="package://ruiyan_rh2_hand_description/urdf/meshes/ruihand6z/fz23_Link.STL"/>
+          <mesh filename="package://ruiyan_rh2_hand_description/meshes/ruihand6z/fz23_Link.STL"/>
         </geometry>
         <material name="">
@@ -241,5 +241,5 @@
         <origin xyz="0 0 0" rpy="0 0 0"/>
         <geometry>
-          <mesh filename="package://ruiyan_rh2_hand_description/urdf/meshes/ruihand6z/fz23_Link.STL"/>
+          <mesh filename="package://ruiyan_rh2_hand_description/meshes/ruihand6z/fz23_Link.STL"/>
         </geometry>
       </collision>
@@ -263,14 +263,14 @@
         <origin xyz="0 0 0" rpy="0 0 0"/>
         <geometry>
-          <mesh filename="package://ruiyan_rh2_hand_description/urdf/meshes/ruihand6z/fz31_Link.STL"/>
-        </geometry>
-        <material name="">
-          <color rgba="0.898039215686275 0.917647058823529 0.929411764705882 1"/>
-        </material>
-      </visual>
-      <collision>
-        <origin xyz="0 0 0" rpy="0 0 0"/>
-        <geometry>
-          <mesh filename="package://ruiyan_rh2_hand_description/urdf/meshes/ruihand6z/fz31_Link.STL"/>
+          <mesh filename="package://ruiyan_rh2_hand_description/meshes/ruihand6z/fz31_Link.STL"/>
+        </geometry>
+        <material name="">
+          <color rgba="0.898039215686275 0.917647058823529 0.929411764705882 1"/>
+        </material>
+      </visual>
+      <collision>
+        <origin xyz="0 0 0" rpy="0 0 0"/>
+        <geometry>
+          <mesh filename="package://ruiyan_rh2_hand_description/meshes/ruihand6z/fz31_Link.STL"/>
         </geometry>
       </collision>
@@ -294,5 +294,5 @@
         <origin xyz="0 0 0" rpy="0 0 0"/>
         <geometry>
-          <mesh filename="package://ruiyan_rh2_hand_description/urdf/meshes/ruihand6z/fz32_Link.STL"/>
+          <mesh filename="package://ruiyan_rh2_hand_description/meshes/ruihand6z/fz32_Link.STL"/>
         </geometry>
         <material name="">
@@ -303,5 +303,5 @@
         <origin xyz="0 0 0" rpy="0 0 0"/>
         <geometry>
-          <mesh filename="package://ruiyan_rh2_hand_description/urdf/meshes/ruihand6z/fz32_Link.STL"/>
+          <mesh filename="package://ruiyan_rh2_hand_description/meshes/ruihand6z/fz32_Link.STL"/>
         </geometry>
       </collision>
@@ -326,5 +326,5 @@
         <origin xyz="0 0 0" rpy="0 0 0"/>
         <geometry>
-          <mesh filename="package://ruiyan_rh2_hand_description/urdf/meshes/ruihand6z/fz33_Link.STL"/>
+          <mesh filename="package://ruiyan_rh2_hand_description/meshes/ruihand6z/fz33_Link.STL"/>
         </geometry>
         <material name="">
@@ -335,5 +335,5 @@
         <origin xyz="0 0 0" rpy="0 0 0"/>
         <geometry>
-          <mesh filename="package://ruiyan_rh2_hand_description/urdf/meshes/ruihand6z/fz33_Link.STL"/>
+          <mesh filename="package://ruiyan_rh2_hand_description/meshes/ruihand6z/fz33_Link.STL"/>
         </geometry>
       </collision>
@@ -357,14 +357,14 @@
         <origin xyz="0 0 0" rpy="0 0 0"/>
         <geometry>
-          <mesh filename="package://ruiyan_rh2_hand_description/urdf/meshes/ruihand6z/fz41_Link.STL"/>
-        </geometry>
-        <material name="">
-          <color rgba="0.898039215686275 0.917647058823529 0.929411764705882 1"/>
-        </material>
-      </visual>
-      <collision>
-        <origin xyz="0 0 0" rpy="0 0 0"/>
-        <geometry>
-          <mesh filename="package://ruiyan_rh2_hand_description/urdf/meshes/ruihand6z/fz41_Link.STL"/>
+          <mesh filename="package://ruiyan_rh2_hand_description/meshes/ruihand6z/fz41_Link.STL"/>
+        </geometry>
+        <material name="">
+          <color rgba="0.898039215686275 0.917647058823529 0.929411764705882 1"/>
+        </material>
+      </visual>
+      <collision>
+        <origin xyz="0 0 0" rpy="0 0 0"/>
+        <geometry>
+          <mesh filename="package://ruiyan_rh2_hand_description/meshes/ruihand6z/fz41_Link.STL"/>
         </geometry>
       </collision>
@@ -388,5 +388,5 @@
         <origin xyz="0 0 0" rpy="0 0 0"/>
         <geometry>
-          <mesh filename="package://ruiyan_rh2_hand_description/urdf/meshes/ruihand6z/fz42_Link.STL"/>
+          <mesh filename="package://ruiyan_rh2_hand_description/meshes/ruihand6z/fz42_Link.STL"/>
         </geometry>
         <material name="">
@@ -397,5 +397,5 @@
         <origin xyz="0 0 0" rpy="0 0 0"/>
         <geometry>
-          <mesh filename="package://ruiyan_rh2_hand_description/urdf/meshes/ruihand6z/fz42_Link.STL"/>
+          <mesh filename="package://ruiyan_rh2_hand_description/meshes/ruihand6z/fz42_Link.STL"/>
         </geometry>
       </collision>
@@ -420,5 +420,5 @@
         <origin xyz="0 0 0" rpy="0 0 0"/>
         <geometry>
-          <mesh filename="package://ruiyan_rh2_hand_description/urdf/meshes/ruihand6z/fz43_Link.STL"/>
+          <mesh filename="package://ruiyan_rh2_hand_description/meshes/ruihand6z/fz43_Link.STL"/>
         </geometry>
         <material name="">
@@ -429,5 +429,5 @@
         <origin xyz="0 0 0" rpy="0 0 0"/>
         <geometry>
-          <mesh filename="package://ruiyan_rh2_hand_description/urdf/meshes/ruihand6z/fz43_Link.STL"/>
+          <mesh filename="package://ruiyan_rh2_hand_description/meshes/ruihand6z/fz43_Link.STL"/>
         </geometry>
       </collision>
@@ -451,14 +451,14 @@
         <origin xyz="0 0 0" rpy="0 0 0"/>
         <geometry>
-          <mesh filename="package://ruiyan_rh2_hand_description/urdf/meshes/ruihand6z/fz51_Link.STL"/>
-        </geometry>
-        <material name="">
-          <color rgba="0.898039215686275 0.917647058823529 0.929411764705882 1"/>
-        </material>
-      </visual>
-      <collision>
-        <origin xyz="0 0 0" rpy="0 0 0"/>
-        <geometry>
-          <mesh filename="package://ruiyan_rh2_hand_description/urdf/meshes/ruihand6z/fz51_Link.STL"/>
+          <mesh filename="package://ruiyan_rh2_hand_description/meshes/ruihand6z/fz51_Link.STL"/>
+        </geometry>
+        <material name="">
+          <color rgba="0.898039215686275 0.917647058823529 0.929411764705882 1"/>
+        </material>
+      </visual>
+      <collision>
+        <origin xyz="0 0 0" rpy="0 0 0"/>
+        <geometry>
+          <mesh filename="package://ruiyan_rh2_hand_description/meshes/ruihand6z/fz51_Link.STL"/>
         </geometry>
       </collision>
@@ -482,5 +482,5 @@
         <origin xyz="0 0 0" rpy="0 0 0"/>
         <geometry>
-          <mesh filename="package://ruiyan_rh2_hand_description/urdf/meshes/ruihand6z/fz52_Link.STL"/>
+          <mesh filename="package://ruiyan_rh2_hand_description/meshes/ruihand6z/fz52_Link.STL"/>
         </geometry>
         <material name="">
@@ -491,5 +491,5 @@
         <origin xyz="0 0 0" rpy="0 0 0"/>
         <geometry>
-          <mesh filename="package://ruiyan_rh2_hand_description/urdf/meshes/ruihand6z/fz52_Link.STL"/>
+          <mesh filename="package://ruiyan_rh2_hand_description/meshes/ruihand6z/fz52_Link.STL"/>
         </geometry>
       </collision>
@@ -514,5 +514,5 @@
         <origin xyz="0 0 0" rpy="0 0 0"/>
         <geometry>
-          <mesh filename="package://ruiyan_rh2_hand_description/urdf/meshes/ruihand6z/fz53_Link.STL"/>
+          <mesh filename="package://ruiyan_rh2_hand_description/meshes/ruihand6z/fz53_Link.STL"/>
         </geometry>
         <material name="">
@@ -523,5 +523,5 @@
         <origin xyz="0 0 0" rpy="0 0 0"/>
         <geometry>
-          <mesh filename="package://ruiyan_rh2_hand_description/urdf/meshes/ruihand6z/fz53_Link.STL"/>
+          <mesh filename="package://ruiyan_rh2_hand_description/meshes/ruihand6z/fz53_Link.STL"/>
         </geometry>
       </collision>
