Commit message: Refactor folder structure to follow ros conventions
Signed-off-by: Baoan Du <baoan.du.xj@renesas.com>

File: urdf/ruiyan_hand_right_macro.xacro (robot description, xacro)
@@ -20,14 +20,14 @@
         <origin xyz="0 0 0" rpy="0 0 0"/>
         <geometry>
-          <mesh filename="package://ruiyan_rh2_hand_description/urdf/meshes/ruihand6y/base_link.STL"/>
-        </geometry>
-        <material name="">
-          <color rgba="0.898039215686275 0.917647058823529 0.929411764705882 1"/>
-        </material>
-      </visual>
-      <collision>
-        <origin xyz="0 0 0" rpy="0 0 0"/>
-        <geometry>
-          <mesh filename="package://ruiyan_rh2_hand_description/urdf/meshes/ruihand6y/base_link.STL"/>
+          <mesh filename="package://ruiyan_rh2_hand_description/meshes/ruihand6y/base_link.STL"/>
+        </geometry>
+        <material name="">
+          <color rgba="0.898039215686275 0.917647058823529 0.929411764705882 1"/>
+        </material>
+      </visual>
+      <collision>
+        <origin xyz="0 0 0" rpy="0 0 0"/>
+        <geometry>
+          <mesh filename="package://ruiyan_rh2_hand_description/meshes/ruihand6y/base_link.STL"/>
         </geometry>
       </collision>
@@ -44,14 +44,14 @@
         <origin xyz="0 0 0" rpy="0 0 0"/>
         <geometry>
-          <mesh filename="package://ruiyan_rh2_hand_description/urdf/meshes/ruihand6y/fy11_Link.STL"/>
-        </geometry>
-        <material name="">
-          <color rgba="0.898039215686275 0.917647058823529 0.929411764705882 1"/>
-        </material>
-      </visual>
-      <collision>
-        <origin xyz="0 0 0" rpy="0 0 0"/>
-        <geometry>
-          <mesh filename="package://ruiyan_rh2_hand_description/urdf/meshes/ruihand6y/fy11_Link.STL"/>
+          <mesh filename="package://ruiyan_rh2_hand_description/meshes/ruihand6y/fy11_Link.STL"/>
+        </geometry>
+        <material name="">
+          <color rgba="0.898039215686275 0.917647058823529 0.929411764705882 1"/>
+        </material>
+      </visual>
+      <collision>
+        <origin xyz="0 0 0" rpy="0 0 0"/>
+        <geometry>
+          <mesh filename="package://ruiyan_rh2_hand_description/meshes/ruihand6y/fy11_Link.STL"/>
         </geometry>
       </collision>
@@ -75,14 +75,14 @@
         <origin xyz="0 0 0" rpy="0 0 0"/>
         <geometry>
-          <mesh filename="package://ruiyan_rh2_hand_description/urdf/meshes/ruihand6y/fy12_Link.STL"/>
-        </geometry>
-        <material name="">
-          <color rgba="0.898039215686275 0.917647058823529 0.929411764705882 1"/>
-        </material>
-      </visual>
-      <collision>
-        <origin xyz="0 0 0" rpy="0 0 0"/>
-        <geometry>
-          <mesh filename="package://ruiyan_rh2_hand_description/urdf/meshes/ruihand6y/fy12_Link.STL"/>
+          <mesh filename="package://ruiyan_rh2_hand_description/meshes/ruihand6y/fy12_Link.STL"/>
+        </geometry>
+        <material name="">
+          <color rgba="0.898039215686275 0.917647058823529 0.929411764705882 1"/>
+        </material>
+      </visual>
+      <collision>
+        <origin xyz="0 0 0" rpy="0 0 0"/>
+        <geometry>
+          <mesh filename="package://ruiyan_rh2_hand_description/meshes/ruihand6y/fy12_Link.STL"/>
         </geometry>
       </collision>
@@ -106,14 +106,14 @@
         <origin xyz="0 0 0" rpy="0 0 0"/>
         <geometry>
-          <mesh filename="package://ruiyan_rh2_hand_description/urdf/meshes/ruihand6y/fy13_Link.STL"/>
-        </geometry>
-        <material name="">
-          <color rgba="0.898039215686275 0.917647058823529 0.929411764705882 1"/>
-        </material>
-      </visual>
-      <collision>
-        <origin xyz="0 0 0" rpy="0 0 0"/>
-        <geometry>
-          <mesh filename="package://ruiyan_rh2_hand_description/urdf/meshes/ruihand6y/fy13_Link.STL"/>
+          <mesh filename="package://ruiyan_rh2_hand_description/meshes/ruihand6y/fy13_Link.STL"/>
+        </geometry>
+        <material name="">
+          <color rgba="0.898039215686275 0.917647058823529 0.929411764705882 1"/>
+        </material>
+      </visual>
+      <collision>
+        <origin xyz="0 0 0" rpy="0 0 0"/>
+        <geometry>
+          <mesh filename="package://ruiyan_rh2_hand_description/meshes/ruihand6y/fy13_Link.STL"/>
         </geometry>
       </collision>
@@ -138,5 +138,5 @@
         <origin xyz="0 0 0" rpy="0 0 0"/>
         <geometry>
-          <mesh filename="package://ruiyan_rh2_hand_description/urdf/meshes/ruihand6y/fy14_Link.STL"/>
+          <mesh filename="package://ruiyan_rh2_hand_description/meshes/ruihand6y/fy14_Link.STL"/>
         </geometry>
         <material name="">
@@ -147,5 +147,5 @@
         <origin xyz="0 0 0" rpy="0 0 0"/>
         <geometry>
-          <mesh filename="package://ruiyan_rh2_hand_description/urdf/meshes/ruihand6y/fy14_Link.STL"/>
+          <mesh filename="package://ruiyan_rh2_hand_description/meshes/ruihand6y/fy14_Link.STL"/>
         </geometry>
       </collision>
@@ -169,14 +169,14 @@
         <origin xyz="0 0 0" rpy="0 0 0"/>
         <geometry>
-          <mesh filename="package://ruiyan_rh2_hand_description/urdf/meshes/ruihand6y/fy21_Link.STL"/>
-        </geometry>
-        <material name="">
-          <color rgba="0.898039215686275 0.917647058823529 0.929411764705882 1"/>
-        </material>
-      </visual>
-      <collision>
-        <origin xyz="0 0 0" rpy="0 0 0"/>
-        <geometry>
-          <mesh filename="package://ruiyan_rh2_hand_description/urdf/meshes/ruihand6y/fy21_Link.STL"/>
+          <mesh filename="package://ruiyan_rh2_hand_description/meshes/ruihand6y/fy21_Link.STL"/>
+        </geometry>
+        <material name="">
+          <color rgba="0.898039215686275 0.917647058823529 0.929411764705882 1"/>
+        </material>
+      </visual>
+      <collision>
+        <origin xyz="0 0 0" rpy="0 0 0"/>
+        <geometry>
+          <mesh filename="package://ruiyan_rh2_hand_description/meshes/ruihand6y/fy21_Link.STL"/>
         </geometry>
       </collision>
@@ -200,5 +200,5 @@
         <origin xyz="0 0 0" rpy="0 0 0"/>
         <geometry>
-          <mesh filename="package://ruiyan_rh2_hand_description/urdf/meshes/ruihand6y/fy22_Link.STL"/>
+          <mesh filename="package://ruiyan_rh2_hand_description/meshes/ruihand6y/fy22_Link.STL"/>
         </geometry>
         <material name="">
@@ -209,5 +209,5 @@
         <origin xyz="0 0 0" rpy="0 0 0"/>
         <geometry>
-          <mesh filename="package://ruiyan_rh2_hand_description/urdf/meshes/ruihand6y/fy22_Link.STL"/>
+          <mesh filename="package://ruiyan_rh2_hand_description/meshes/ruihand6y/fy22_Link.STL"/>
         </geometry>
       </collision>
@@ -232,5 +232,5 @@
         <origin xyz="0 0 0" rpy="0 0 0"/>
         <geometry>
-          <mesh filename="package://ruiyan_rh2_hand_description/urdf/meshes/ruihand6y/fy23_Link.STL"/>
+          <mesh filename="package://ruiyan_rh2_hand_description/meshes/ruihand6y/fy23_Link.STL"/>
         </geometry>
         <material name="">
@@ -241,5 +241,5 @@
         <origin xyz="0 0 0" rpy="0 0 0"/>
         <geometry>
-          <mesh filename="package://ruiyan_rh2_hand_description/urdf/meshes/ruihand6y/fy23_Link.STL"/>
+          <mesh filename="package://ruiyan_rh2_hand_description/meshes/ruihand6y/fy23_Link.STL"/>
         </geometry>
       </collision>
@@ -263,14 +263,14 @@
         <origin xyz="0 0 0" rpy="0 0 0"/>
         <geometry>
-          <mesh filename="package://ruiyan_rh2_hand_description/urdf/meshes/ruihand6y/fy31_Link.STL"/>
-        </geometry>
-        <material name="">
-          <color rgba="0.898039215686275 0.917647058823529 0.929411764705882 1"/>
-        </material>
-      </visual>
-      <collision>
-        <origin xyz="0 0 0" rpy="0 0 0"/>
-        <geometry>
-          <mesh filename="package://ruiyan_rh2_hand_description/urdf/meshes/ruihand6y/fy31_Link.STL"/>
+          <mesh filename="package://ruiyan_rh2_hand_description/meshes/ruihand6y/fy31_Link.STL"/>
+        </geometry>
+        <material name="">
+          <color rgba="0.898039215686275 0.917647058823529 0.929411764705882 1"/>
+        </material>
+      </visual>
+      <collision>
+        <origin xyz="0 0 0" rpy="0 0 0"/>
+        <geometry>
+          <mesh filename="package://ruiyan_rh2_hand_description/meshes/ruihand6y/fy31_Link.STL"/>
         </geometry>
       </collision>
@@ -294,5 +294,5 @@
         <origin xyz="0 0 0" rpy="0 0 0"/>
         <geometry>
-          <mesh filename="package://ruiyan_rh2_hand_description/urdf/meshes/ruihand6y/fy32_Link.STL"/>
+          <mesh filename="package://ruiyan_rh2_hand_description/meshes/ruihand6y/fy32_Link.STL"/>
         </geometry>
         <material name="">
@@ -303,5 +303,5 @@
         <origin xyz="0 0 0" rpy="0 0 0"/>
         <geometry>
-          <mesh filename="package://ruiyan_rh2_hand_description/urdf/meshes/ruihand6y/fy32_Link.STL"/>
+          <mesh filename="package://ruiyan_rh2_hand_description/meshes/ruihand6y/fy32_Link.STL"/>
         </geometry>
       </collision>
@@ -326,5 +326,5 @@
         <origin xyz="0 0 0" rpy="0 0 0"/>
         <geometry>
-          <mesh filename="package://ruiyan_rh2_hand_description/urdf/meshes/ruihand6y/fy33_Link.STL"/>
+          <mesh filename="package://ruiyan_rh2_hand_description/meshes/ruihand6y/fy33_Link.STL"/>
         </geometry>
         <material name="">
@@ -335,5 +335,5 @@
         <origin xyz="0 0 0" rpy="0 0 0"/>
         <geometry>
-          <mesh filename="package://ruiyan_rh2_hand_description/urdf/meshes/ruihand6y/fy33_Link.STL"/>
+          <mesh filename="package://ruiyan_rh2_hand_description/meshes/ruihand6y/fy33_Link.STL"/>
         </geometry>
       </collision>
@@ -357,14 +357,14 @@
         <origin xyz="0 0 0" rpy="0 0 0"/>
         <geometry>
-          <mesh filename="package://ruiyan_rh2_hand_description/urdf/meshes/ruihand6y/fy41_Link.STL"/>
-        </geometry>
-        <material name="">
-          <color rgba="0.898039215686275 0.917647058823529 0.929411764705882 1"/>
-        </material>
-      </visual>
-      <collision>
-        <origin xyz="0 0 0" rpy="0 0 0"/>
-        <geometry>
-          <mesh filename="package://ruiyan_rh2_hand_description/urdf/meshes/ruihand6y/fy41_Link.STL"/>
+          <mesh filename="package://ruiyan_rh2_hand_description/meshes/ruihand6y/fy41_Link.STL"/>
+        </geometry>
+        <material name="">
+          <color rgba="0.898039215686275 0.917647058823529 0.929411764705882 1"/>
+        </material>
+      </visual>
+      <collision>
+        <origin xyz="0 0 0" rpy="0 0 0"/>
+        <geometry>
+          <mesh filename="package://ruiyan_rh2_hand_description/meshes/ruihand6y/fy41_Link.STL"/>
         </geometry>
       </collision>
@@ -388,5 +388,5 @@
         <origin xyz="0 0 0" rpy="0 0 0"/>
         <geometry>
-          <mesh filename="package://ruiyan_rh2_hand_description/urdf/meshes/ruihand6y/fy42_Link.STL"/>
+          <mesh filename="package://ruiyan_rh2_hand_description/meshes/ruihand6y/fy42_Link.STL"/>
         </geometry>
         <material name="">
@@ -397,5 +397,5 @@
         <origin xyz="0 0 0" rpy="0 0 0"/>
         <geometry>
-          <mesh filename="package://ruiyan_rh2_hand_description/urdf/meshes/ruihand6y/fy42_Link.STL"/>
+          <mesh filename="package://ruiyan_rh2_hand_description/meshes/ruihand6y/fy42_Link.STL"/>
         </geometry>
       </collision>
@@ -420,5 +420,5 @@
         <origin xyz="0 0 0" rpy="0 0 0"/>
         <geometry>
-          <mesh filename="package://ruiyan_rh2_hand_description/urdf/meshes/ruihand6y/fy43_Link.STL"/>
+          <mesh filename="package://ruiyan_rh2_hand_description/meshes/ruihand6y/fy43_Link.STL"/>
         </geometry>
         <material name="">
@@ -429,5 +429,5 @@
         <origin xyz="0 0 0" rpy="0 0 0"/>
         <geometry>
-          <mesh filename="package://ruiyan_rh2_hand_description/urdf/meshes/ruihand6y/fy43_Link.STL"/>
+          <mesh filename="package://ruiyan_rh2_hand_description/meshes/ruihand6y/fy43_Link.STL"/>
         </geometry>
       </collision>
@@ -451,14 +451,14 @@
         <origin xyz="0 0 0" rpy="0 0 0"/>
         <geometry>
-          <mesh filename="package://ruiyan_rh2_hand_description/urdf/meshes/ruihand6y/fy51_Link.STL"/>
-        </geometry>
-        <material name="">
-          <color rgba="0.898039215686275 0.917647058823529 0.929411764705882 1"/>
-        </material>
-      </visual>
-      <collision>
-        <origin xyz="0 0 0" rpy="0 0 0"/>
-        <geometry>
-          <mesh filename="package://ruiyan_rh2_hand_description/urdf/meshes/ruihand6y/fy51_Link.STL"/>
+          <mesh filename="package://ruiyan_rh2_hand_description/meshes/ruihand6y/fy51_Link.STL"/>
+        </geometry>
+        <material name="">
+          <color rgba="0.898039215686275 0.917647058823529 0.929411764705882 1"/>
+        </material>
+      </visual>
+      <collision>
+        <origin xyz="0 0 0" rpy="0 0 0"/>
+        <geometry>
+          <mesh filename="package://ruiyan_rh2_hand_description/meshes/ruihand6y/fy51_Link.STL"/>
         </geometry>
       </collision>
@@ -482,5 +482,5 @@
         <origin xyz="0 0 0" rpy="0 0 0"/>
         <geometry>
-          <mesh filename="package://ruiyan_rh2_hand_description/urdf/meshes/ruihand6y/fy52_Link.STL"/>
+          <mesh filename="package://ruiyan_rh2_hand_description/meshes/ruihand6y/fy52_Link.STL"/>
         </geometry>
         <material name="">
@@ -491,5 +491,5 @@
         <origin xyz="0 0 0" rpy="0 0 0"/>
         <geometry>
-          <mesh filename="package://ruiyan_rh2_hand_description/urdf/meshes/ruihand6y/fy52_Link.STL"/>
+          <mesh filename="package://ruiyan_rh2_hand_description/meshes/ruihand6y/fy52_Link.STL"/>
         </geometry>
       </collision>
@@ -514,5 +514,5 @@
         <origin xyz="0 0 0" rpy="0 0 0"/>
         <geometry>
-          <mesh filename="package://ruiyan_rh2_hand_description/urdf/meshes/ruihand6y/fy53_Link.STL"/>
+          <mesh filename="package://ruiyan_rh2_hand_description/meshes/ruihand6y/fy53_Link.STL"/>
         </geometry>
         <material name="">
@@ -523,5 +523,5 @@
         <origin xyz="0 0 0" rpy="0 0 0"/>
         <geometry>
-          <mesh filename="package://ruiyan_rh2_hand_description/urdf/meshes/ruihand6y/fy53_Link.STL"/>
+          <mesh filename="package://ruiyan_rh2_hand_description/meshes/ruihand6y/fy53_Link.STL"/>
         </geometry>
       </collision>
