Commit message: Avoid base link naming conflict in multi robot setup
Signed-off-by: Baoan Du <baoan.du.xj@renesas.com>

File: urdf/ruiyan_hand_left_macro.xacro (robot description, xacro)
@@ -7,8 +7,8 @@
       <xacro:insert_block name="origin" />
       <parent link="${parent}"/>
-      <child link="${prefix}base_link"/>
+      <child link="${prefix}hand_base_link"/>
     </joint>
     <!-- Base link -->
-    <link name="${prefix}base_link">
+    <link name="${prefix}hand_base_link">
       <inertial>
         <origin xyz="-0.00261509912067082 -0.00202384901005411 0.0609899196930254" rpy="0 0 0"/>
@@ -59,5 +59,5 @@
     <joint name="${prefix}thumb_proximal_yaw_joint" type="revolute">
       <origin xyz="0.0135 -0.022 0.0398" rpy="0 0 1.5708"/>
-      <parent link="${prefix}base_link"/>
+      <parent link="${prefix}hand_base_link"/>
       <child link="${prefix}fz11_Link"/>
       <axis xyz="0 0 1"/>
@@ -184,5 +184,5 @@
     <joint name="${prefix}index_proximal_joint" type="revolute">
       <origin xyz="-0.0035 -0.029833 0.11095" rpy="3.1416 1.4923 1.5708"/>
-      <parent link="${prefix}base_link"/>
+      <parent link="${prefix}hand_base_link"/>
       <child link="${prefix}fz21_Link"/>
       <axis xyz="0 0 -1"/>
@@ -278,5 +278,5 @@
     <joint name="${prefix}middle_proximal_joint" type="revolute">
       <origin xyz="-0.0035 -0.009945 0.112" rpy="3.1416 1.5446 1.5708"/>
-      <parent link="${prefix}base_link"/>
+      <parent link="${prefix}hand_base_link"/>
       <child link="${prefix}fz31_Link"/>
       <axis xyz="0 0 -1"/>
@@ -372,5 +372,5 @@
     <joint name="${prefix}ring_proximal_joint" type="revolute">
       <origin xyz="-0.0035 0.009945 0.11099" rpy="0 1.5446 -1.5708"/>
-      <parent link="${prefix}base_link"/>
+      <parent link="${prefix}hand_base_link"/>
       <child link="${prefix}fz41_Link"/>
       <axis xyz="0 0 -1"/>
@@ -466,5 +466,5 @@
     <joint name="${prefix}pinky_proximal_joint" type="revolute">
       <origin xyz="-0.0035 0.029624 0.10795" rpy="0 1.4923 -1.5708"/>
-      <parent link="${prefix}base_link"/>
+      <parent link="${prefix}hand_base_link"/>
       <child link="${prefix}fz51_Link"/>
       <axis xyz="0 0 -1"/>

File: urdf/ruiyan_hand_right_macro.xacro (robot description, xacro)
@@ -7,8 +7,8 @@
       <xacro:insert_block name="origin" />
       <parent link="${parent}"/>
-      <child link="${prefix}base_link"/>
+      <child link="${prefix}hand_base_link"/>
     </joint>
     <!-- Base link -->
-    <link name="${prefix}base_link">
+    <link name="${prefix}hand_base_link">
       <inertial>
         <origin xyz="-0.00354104285456125 0.00204598885782099 0.0605396757269698" rpy="0 0 0"/>
@@ -59,5 +59,5 @@
     <joint name="${prefix}thumb_proximal_yaw_joint" type="revolute">
       <origin xyz="0.0135 0.022 0.0398" rpy="0 0 1.5708"/>
-      <parent link="${prefix}base_link"/>
+      <parent link="${prefix}hand_base_link"/>
       <child link="${prefix}fy11_Link"/>
       <axis xyz="0 0 -1"/>
@@ -184,5 +184,5 @@
     <joint name="${prefix}index_proximal_joint" type="revolute">
       <origin xyz="-0.0035 0.029833 0.11095" rpy="0 -1.4923 1.5708"/>
-      <parent link="${prefix}base_link"/>
+      <parent link="${prefix}hand_base_link"/>
       <child link="${prefix}fy21_Link"/>
       <axis xyz="0 0 -1"/>
@@ -278,5 +278,5 @@
     <joint name="${prefix}middle_proximal_joint" type="revolute">
       <origin xyz="-0.0035 0.009945 0.112" rpy="0 -1.5446 1.5708"/>
-      <parent link="${prefix}base_link"/>
+      <parent link="${prefix}hand_base_link"/>
       <child link="${prefix}fy31_Link"/>
       <axis xyz="0 0 -1"/>
@@ -372,5 +372,5 @@
     <joint name="${prefix}ring_proximal_joint" type="revolute">
       <origin xyz="-0.0035 -0.009945 0.11099" rpy="3.1416 -1.5446 -1.5708"/>
-      <parent link="${prefix}base_link"/>
+      <parent link="${prefix}hand_base_link"/>
       <child link="${prefix}fy41_Link"/>
       <axis xyz="0 0 -1"/>
@@ -466,5 +466,5 @@
     <joint name="${prefix}pinky_proximal_joint" type="revolute">
       <origin xyz="-0.0035 -0.029624 0.10795" rpy="3.1416 -1.4923 -1.5708"/>
-      <parent link="${prefix}base_link"/>
+      <parent link="${prefix}hand_base_link"/>
       <child link="${prefix}fy51_Link"/>
       <axis xyz="0 0 -1"/>

Commit message: Add TCP link and joint for three-finger grasp in left and right hand macros
Further calibration on physical hand is required.

Signed-off-by: Baoan Du <baoan.du.xj@renesas.com>

File: urdf/ruiyan_hand_left_macro.xacro (robot description, xacro)
@@ -534,4 +534,18 @@
       <limit lower="0" upper="0" effort="1" velocity="0.5"/>
     </joint>
+    <!-- Three-finger grasp TCP -->
+    <link name="${prefix}tcp">
+      <inertial>
+        <origin xyz="0 0 0" rpy="0 0 0"/>
+        <mass value="1e-06"/>
+        <inertia ixx="1e-09" ixy="0" ixz="0" iyy="1e-09" iyz="0" izz="1e-09"/>
+      </inertial>
+    </link>
+    <joint name="${prefix}tcp_joint" type="fixed">
+      <!-- Measured tcp position relative to base frame -->
+      <origin xyz="0.075 -0.020 0.130" rpy="0 0.785398 0"/>
+      <parent link="${prefix}hand_base_link"/>
+      <child link="${prefix}tcp"/>
+    </joint>
   </xacro:macro>
 </robot>

File: urdf/ruiyan_hand_right_macro.xacro (robot description, xacro)
@@ -534,4 +534,18 @@
       <limit lower="0" upper="0" effort="1" velocity="0.5"/>
     </joint>
+    <!-- Three-finger grasp TCP -->
+    <link name="${prefix}tcp">
+      <inertial>
+        <origin xyz="0 0 0" rpy="0 0 0"/>
+        <mass value="1e-06"/>
+        <inertia ixx="1e-09" ixy="0" ixz="0" iyy="1e-09" iyz="0" izz="1e-09"/>
+      </inertial>
+    </link>
+    <joint name="${prefix}tcp_joint" type="fixed">
+      <!-- Measured tcp position relative to base frame -->
+      <origin xyz="0.075 0.020 0.130" rpy="0 0.785398 0"/>
+      <parent link="${prefix}hand_base_link"/>
+      <child link="${prefix}tcp"/>
+    </joint>
   </xacro:macro>
 </robot>

Commit message: Add velocity limitation for suitable with ros2 control flow
Signed-off-by: Dat Nguyen <dat.nguyen.dn@bp.renesas.com>

File: urdf/ruiyan_hand_left_macro.xacro (robot description, xacro)
@@ -62,5 +62,5 @@
       <child link="${prefix}fz11_Link"/>
       <axis xyz="0 0 1"/>
-      <limit lower="0" upper="2.356" effort="1" velocity="0.5"/>
+      <limit lower="0" upper="2.356" effort="1" velocity="11.78"/>
     </joint>
     <!-- Thumb proximal pitch -->
@@ -93,5 +93,5 @@
       <child link="${prefix}fz12_Link"/>
       <axis xyz="0 0 -1"/>
-      <limit lower="0" upper="0.698" effort="1" velocity="0.5"/>
+      <limit lower="0" upper="0.698" effort="1" velocity="3.49"/>
     </joint>
     <!-- Thumb intermediate -->
@@ -124,5 +124,5 @@
       <child link="${prefix}fz13_Link"/>
       <axis xyz="0 0 -1"/>
-      <limit lower="0" upper="1.169" effort="1" velocity="0.5"/>
+      <limit lower="0" upper="1.169" effort="1" velocity="5.845"/>
       <mimic joint="${prefix}thumb_proximal_pitch_joint" multiplier="1.334" offset="0"/>
     </joint>
@@ -156,5 +156,5 @@
       <child link="${prefix}fz14_Link"/>
       <axis xyz="0 0 -1"/>
-      <limit lower="0" upper="0" effort="1" velocity="0.5"/>
+      <limit lower="0" upper="0" effort="1" velocity="3.0"/>
     </joint>
     <!-- Index finger proximal -->
@@ -187,5 +187,5 @@
       <child link="${prefix}fz21_Link"/>
       <axis xyz="0 0 -1"/>
-      <limit lower="0" upper="1.518" effort="1" velocity="0.5"/>
+      <limit lower="0" upper="1.518" effort="1" velocity="7.59"/>
     </joint>
     <!-- Index finger intermediate -->
@@ -218,5 +218,5 @@
       <child link="${prefix}fz22_Link"/>
       <axis xyz="0 0 -1"/>
-      <limit lower="0" upper="1.623" effort="1" velocity="0.5"/>
+      <limit lower="0" upper="1.623" effort="1" velocity="8.115"/>
       <mimic joint="${prefix}index_proximal_joint" multiplier="1.06399" offset="-0.04545"/>
     </joint>
@@ -250,5 +250,5 @@
       <child link="${prefix}fz23_Link"/>
       <axis xyz="0 0 -1"/>
-      <limit lower="0" upper="0" effort="1" velocity="0.5"/>
+      <limit lower="0" upper="0" effort="1" velocity="3.0"/>
     </joint>
     <!-- Middle finger proximal -->
@@ -281,5 +281,5 @@
       <child link="${prefix}fz31_Link"/>
       <axis xyz="0 0 -1"/>
-      <limit lower="0" upper="1.571" effort="1" velocity="0.5"/>
+      <limit lower="0" upper="1.571" effort="1" velocity="7.855"/>
     </joint>
     <!-- Middle finger intermediate -->
@@ -312,5 +312,5 @@
       <child link="${prefix}fz32_Link"/>
       <axis xyz="0 0 -1"/>
-      <limit lower="0" upper="1.641" effort="1" velocity="0.5"/>
+      <limit lower="0" upper="1.641" effort="1" velocity="8.205"/>
       <mimic joint="${prefix}middle_proximal_joint" multiplier="1.06399" offset="-0.04545"/>
     </joint>
@@ -344,5 +344,5 @@
       <child link="${prefix}fz33_Link"/>
       <axis xyz="0 0 -1"/>
-      <limit lower="0" upper="0" effort="1" velocity="0.5"/>
+      <limit lower="0" upper="0" effort="1" velocity="3.0"/>
     </joint>
     <!-- Ring finger proximal -->
@@ -375,5 +375,5 @@
       <child link="${prefix}fz41_Link"/>
       <axis xyz="0 0 -1"/>
-      <limit lower="0" upper="1.571" effort="1" velocity="0.5"/>
+      <limit lower="0" upper="1.571" effort="1" velocity="7.855"/>
     </joint>
     <!-- Ring finger intermediate -->
@@ -406,5 +406,5 @@
       <child link="${prefix}fz42_Link"/>
       <axis xyz="0 0 -1"/>
-      <limit lower="0" upper="1.658" effort="1" velocity="0.5"/>
+      <limit lower="0" upper="1.658" effort="1" velocity="8.29"/>
       <mimic joint="${prefix}ring_proximal_joint" multiplier="1.06399" offset="-0.04545"/>
     </joint>
@@ -438,5 +438,5 @@
       <child link="${prefix}fz43_Link"/>
       <axis xyz="0 0 -1"/>
-      <limit lower="0" upper="0" effort="1" velocity="0.5"/>
+      <limit lower="0" upper="0" effort="1" velocity="3.0"/>
     </joint>
     <!-- Pinky finger proximal -->
@@ -469,5 +469,5 @@
       <child link="${prefix}fz51_Link"/>
       <axis xyz="0 0 -1"/>
-      <limit lower="0" upper="1.545" effort="1" velocity="0.5"/>
+      <limit lower="0" upper="1.545" effort="1" velocity="7.725"/>
     </joint>
     <!-- Pinky finger intermediate -->
@@ -500,5 +500,5 @@
       <child link="${prefix}fz52_Link"/>
       <axis xyz="0 0 -1"/>
-      <limit lower="0" upper="1.658" effort="1" velocity="0.5"/>
+      <limit lower="0" upper="1.658" effort="1" velocity="8.29"/>
       <mimic joint="${prefix}pinky_proximal_joint" multiplier="1.06399" offset="-0.04545"/>
     </joint>
@@ -532,5 +532,5 @@
       <child link="${prefix}fz53_Link"/>
       <axis xyz="0 0 -1"/>
-      <limit lower="0" upper="0" effort="1" velocity="0.5"/>
+      <limit lower="0" upper="0" effort="1" velocity="0"/>
     </joint>
     <!-- Three-finger grasp TCP -->

File: urdf/ruiyan_hand_right_macro.xacro (robot description, xacro)
@@ -62,5 +62,5 @@
       <child link="${prefix}fy11_Link"/>
       <axis xyz="0 0 -1"/>
-      <limit lower="0" upper="2.356" effort="1" velocity="0.5"/>
+      <limit lower="0" upper="2.356" effort="1" velocity="11.78"/>
     </joint>
     <!-- Thumb proximal pitch -->
@@ -93,5 +93,5 @@
       <child link="${prefix}fy12_Link"/>
       <axis xyz="0 0 1"/>
-      <limit lower="0" upper="0.698" effort="1" velocity="0.5"/>
+      <limit lower="0" upper="0.698" effort="1" velocity="3.49"/>
     </joint>
     <!-- Thumb intermediate -->
@@ -124,5 +124,5 @@
       <child link="${prefix}fy13_Link"/>
       <axis xyz="0 0 1"/>
-      <limit lower="0" upper="1.169" effort="1" velocity="0.5"/>
+      <limit lower="0" upper="1.169" effort="1" velocity="5.845"/>
       <mimic joint="${prefix}thumb_proximal_pitch_joint" multiplier="1.334" offset="0"/>
     </joint>
@@ -187,5 +187,5 @@
       <child link="${prefix}fy21_Link"/>
       <axis xyz="0 0 -1"/>
-      <limit lower="0" upper="1.518" effort="1" velocity="0.5"/>
+      <limit lower="0" upper="1.518" effort="1" velocity="7.59"/>
     </joint>
     <!-- Index finger intermediate -->
@@ -218,5 +218,5 @@
       <child link="${prefix}fy22_Link"/>
       <axis xyz="0 0 -1"/>
-      <limit lower="0" upper="1.623" effort="1" velocity="0.5"/>
+      <limit lower="0" upper="1.623" effort="1" velocity="8.115"/>
       <mimic joint="${prefix}index_proximal_joint" multiplier="1.06399" offset="-0.04545"/>
     </joint>
@@ -281,5 +281,5 @@
       <child link="${prefix}fy31_Link"/>
       <axis xyz="0 0 -1"/>
-      <limit lower="0" upper="1.571" effort="1" velocity="0.5"/>
+      <limit lower="0" upper="1.571" effort="1" velocity="7.855"/>
     </joint>
     <!-- Middle finger intermediate -->
@@ -312,5 +312,5 @@
       <child link="${prefix}fy32_Link"/>
       <axis xyz="0 0 -1"/>
-      <limit lower="0" upper="1.641" effort="1" velocity="0.5"/>
+      <limit lower="0" upper="1.641" effort="1" velocity="8.205"/>
       <mimic joint="${prefix}middle_proximal_joint" multiplier="1.06399" offset="-0.04545"/>
     </joint>
@@ -375,5 +375,5 @@
       <child link="${prefix}fy41_Link"/>
       <axis xyz="0 0 -1"/>
-      <limit lower="0" upper="1.571" effort="1" velocity="0.5"/>
+      <limit lower="0" upper="1.571" effort="1" velocity="7.855"/>
     </joint>
     <!-- Ring finger intermediate -->
@@ -406,5 +406,5 @@
       <child link="${prefix}fy42_Link"/>
       <axis xyz="0 0 -1"/>
-      <limit lower="0" upper="1.658" effort="1" velocity="0.5"/>
+      <limit lower="0" upper="1.658" effort="1" velocity="8.29"/>
       <mimic joint="${prefix}ring_proximal_joint" multiplier="1.06399" offset="-0.04545"/>
     </joint>
@@ -469,5 +469,5 @@
       <child link="${prefix}fy51_Link"/>
       <axis xyz="0 0 -1"/>
-      <limit lower="0" upper="1.545" effort="1" velocity="0.5"/>
+      <limit lower="0" upper="1.545" effort="1" velocity="7.725"/>
     </joint>
     <!-- Pinky finger intermediate -->
@@ -500,5 +500,5 @@
       <child link="${prefix}fy52_Link"/>
       <axis xyz="0 0 -1"/>
-      <limit lower="0" upper="1.658" effort="1" velocity="0.5"/>
+      <limit lower="0" upper="1.658" effort="1" velocity="8.29"/>
       <mimic joint="${prefix}pinky_proximal_joint" multiplier="1.06399" offset="-0.04545"/>
     </joint>

Commit message: Fix the type of last joint of fingers
Signed-off-by: Dat Nguyen <dat.nguyen.dn@bp.renesas.com>

File: urdf/ruiyan_hand_left_macro.xacro (robot description, xacro)
@@ -151,10 +151,9 @@
       </collision>
     </link>
-    <joint name="${prefix}fz14" type="revolute">
+    <joint name="${prefix}fz14" type="fixed">
       <origin xyz="-0.036284 0.0268 0" rpy="-0.3665 -1.5708 0"/>
       <parent link="${prefix}fz13_Link"/>
       <child link="${prefix}fz14_Link"/>
       <axis xyz="0 0 -1"/>
-      <limit lower="0" upper="0" effort="1" velocity="3.0"/>
     </joint>
     <!-- Index finger proximal -->
@@ -245,10 +244,9 @@
       </collision>
     </link>
-    <joint name="${prefix}fz23" type="revolute">
+    <joint name="${prefix}fz23" type="fixed">
       <origin xyz="-0.043692 0.011217 0" rpy="1.5708 1.5695 -1.5543"/>
       <parent link="${prefix}fz22_Link"/>
       <child link="${prefix}fz23_Link"/>
       <axis xyz="0 0 -1"/>
-      <limit lower="0" upper="0" effort="1" velocity="3.0"/>
     </joint>
     <!-- Middle finger proximal -->
@@ -339,10 +337,9 @@
       </collision>
     </link>
-    <joint name="${prefix}fz33" type="revolute">
+    <joint name="${prefix}fz33" type="fixed">
       <origin xyz="-0.043641 0.01141 0" rpy="1.5708 1.5705 -1.5587"/>
       <parent link="${prefix}fz32_Link"/>
       <child link="${prefix}fz33_Link"/>
       <axis xyz="0 0 -1"/>
-      <limit lower="0" upper="0" effort="1" velocity="3.0"/>
     </joint>
     <!-- Ring finger proximal -->
@@ -433,10 +430,9 @@
       </collision>
     </link>
-    <joint name="${prefix}fz43" type="revolute">
+    <joint name="${prefix}fz43" type="fixed">
       <origin xyz="-0.043692 0.011217 0" rpy="-1.5708 1.5704 1.5873"/>
       <parent link="${prefix}fz42_Link"/>
       <child link="${prefix}fz43_Link"/>
       <axis xyz="0 0 -1"/>
-      <limit lower="0" upper="0" effort="1" velocity="3.0"/>
     </joint>
     <!-- Pinky finger proximal -->
@@ -527,10 +523,9 @@
       </collision>
     </link>
-    <joint name="${prefix}fz53" type="revolute">
+    <joint name="${prefix}fz53" type="fixed">
       <origin xyz="-0.043691 0.011217 0" rpy="-1.5708 1.5695 1.5873"/>
       <parent link="${prefix}fz52_Link"/>
       <child link="${prefix}fz53_Link"/>
       <axis xyz="0 0 -1"/>
-      <limit lower="0" upper="0" effort="1" velocity="0"/>
     </joint>
     <!-- Three-finger grasp TCP -->

File: urdf/ruiyan_hand_right_macro.xacro (robot description, xacro)
@@ -151,10 +151,9 @@
       </collision>
     </link>
-    <joint name="${prefix}fy14" type="revolute">
+    <joint name="${prefix}fy14" type="fixed">
       <origin xyz="0.036284 0.0268 0" rpy="-0.36834 1.5708 0"/>
       <parent link="${prefix}fy13_Link"/>
       <child link="${prefix}fy14_Link"/>
       <axis xyz="0 0 1"/>
-      <limit lower="0" upper="0" effort="1" velocity="0.5"/>
     </joint>
     <!-- Index finger proximal -->
@@ -245,10 +244,9 @@
       </collision>
     </link>
-    <joint name="${prefix}fy23" type="revolute">
+    <joint name="${prefix}fy23" type="fixed">
       <origin xyz="0.043692 -0.011217 0" rpy="-1.5708 1.5695 -1.5543"/>
       <parent link="${prefix}fy22_Link"/>
       <child link="${prefix}fy23_Link"/>
       <axis xyz="0 0 -1"/>
-      <limit lower="0" upper="0" effort="1" velocity="0.5"/>
     </joint>
     <!-- Middle finger proximal -->
@@ -339,10 +337,9 @@
       </collision>
     </link>
-    <joint name="${prefix}fy33" type="revolute">
+    <joint name="${prefix}fy33" type="fixed">
       <origin xyz="0.043641 -0.01141 0" rpy="-1.5708 1.5705 -1.5587"/>
       <parent link="${prefix}fy32_Link"/>
       <child link="${prefix}fy33_Link"/>
       <axis xyz="0 0 -1"/>
-      <limit lower="0" upper="0" effort="1" velocity="0.5"/>
     </joint>
     <!-- Ring finger proximal -->
@@ -433,10 +430,9 @@
       </collision>
     </link>
-    <joint name="${prefix}fy43" type="revolute">
+    <joint name="${prefix}fy43" type="fixed">
       <origin xyz="0.043692 -0.011217 0" rpy="1.5708 1.5704 1.5873"/>
       <parent link="${prefix}fy42_Link"/>
       <child link="${prefix}fy43_Link"/>
       <axis xyz="0 0 -1"/>
-      <limit lower="0" upper="0" effort="1" velocity="0.5"/>
     </joint>
     <!-- Pinky finger proximal -->
@@ -527,10 +523,9 @@
       </collision>
     </link>
-    <joint name="${prefix}fy53" type="revolute">
+    <joint name="${prefix}fy53" type="fixed">
       <origin xyz="0.043691 -0.011217 0" rpy="1.5708 1.5695 1.5873"/>
       <parent link="${prefix}fy52_Link"/>
       <child link="${prefix}fy53_Link"/>
       <axis xyz="0 0 -1"/>
-      <limit lower="0" upper="0" effort="1" velocity="0.5"/>
     </joint>
     <!-- Three-finger grasp TCP -->
